File: Pressure-Controlled-Power-Outlet-control-PCB SMD/Pressure-Controlled-Power-Outlet-control-PCB.kicad_sch (KiCad schematic)
At the start: 47 parts, among them J1 pressure sensor, J2 1017514, J3 I2C0 Connector, J4 SPI1 Connector, J5 FanA 5V/24V, J6 FanB 5V/24V, K1 T9GV5L24-24, K2 T9GV5L24-24, M1 Fan_4pin, M2 Fan_4pin, Q1 2N3906, Q2 IRF540N, Q3 IRF540N, Q4 2N3906, Q5 2N3904, Q6 2N3904, Q7 2N3904, Q8 2N3904, U1 Pico, U2 LM324, U3 LF50_TO220

Commit message: make a quick version that has some SMD for pick and place
Parts:
- C2: footprint Capacitor_THT:CP_Radial_D5.0mm_P2.00mm -> Capacitor_SMD:C_1206_3216Metric
- Q2, Q3: footprint Package_TO_SOT_THT:TO-220-3_Vertical -> Package_TO_SOT_SMD:SOT-23-3
- Q5, Q6, Q7, Q8: footprint Package_TO_SOT_THT:TO-92_Inline -> Package_TO_SOT_SMD:SOT-23-3
- R1, R10, R11, R12, R13, R14, R15, R16, R17, R2, R3, R4, R5, R6, R7, R8, R9: footprint Resistor_THT:R_Axial_DIN0207_L6.3mm_D2.5mm_P2.54mm_Vertical -> Resistor_SMD:R_0402_1005Metric
- U2: footprint (none) -> Package_SO:SOIC-14_3.9x8.7mm_P1.27mm
- U2: footprint Package_DIP:DIP-14_W7.62mm_LongPads -> Package_SO:SOIC-14_3.9x8.7mm_P1.27mm
Changed lines of the file:
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@@
       (effects (font (size 1.27 1.27)))
     )
-    (property "Footprint" "Resistor_THT:R_Axial_DIN0207_L6.3mm_D2.5mm_P2.54mm_Vertical" (at 172.72 92.71 0)
+    (property "Footprint" "Resistor_SMD:R_0402_1005Metric" (at 172.72 92.71 0)
       (effects (font (size 1.27 1.27)) hide)
     )
@@
       (effects (font (size 1.27 1.27)) (justify left))
     )
-    (property "Footprint" "Package_TO_SOT_THT:TO-220-3_Vertical" (at 227.33 127.635 0)
+    (property "Footprint" "Package_TO_SOT_SMD:SOT-23-3" (at 227.33 127.635 0)
       (effects (font (size 1.27 1.27) italic) (justify left) hide)
     )
@@
       (effects (font (size 1.27 1.27)) (justify left))
     )
-    (property "Footprint" "Resistor_THT:R_Axial_DIN0207_L6.3mm_D2.5mm_P2.54mm_Vertical" (at 121.92 170.18 0)
+    (property "Footprint" "Resistor_SMD:R_0402_1005Metric" (at 121.92 170.18 0)
       (effects (font (size 1.27 1.27)) hide)
     )
@@
       (effects (font (size 1.27 1.27)) (justify right))
     )
-    (property "Footprint" "Resistor_THT:R_Axial_DIN0207_L6.3mm_D2.5mm_P2.54mm_Vertical" (at 219.71 46.99 0)
+    (property "Footprint" "Resistor_SMD:R_0402_1005Metric" (at 219.71 46.99 0)
       (effects (font (size 1.27 1.27)) hide)
     )
@@
       (effects (font (size 1.27 1.27)) (justify left))
     )
-    (property "Footprint" "Package_TO_SOT_THT:TO-220-3_Vertical" (at 227.33 100.965 0)
+    (property "Footprint" "Package_TO_SOT_SMD:SOT-23-3" (at 227.33 100.965 0)
       (effects (font (size 1.27 1.27) italic) (justify left) hide)
     )
@@
       (effects (font (size 1.27 1.27)) (justify left))
     )
-    (property "Footprint" "Package_TO_SOT_THT:TO-92_Inline" (at 138.43 36.195 0)
+    (property "Footprint" "Package_TO_SOT_SMD:SOT-23-3" (at 138.43 36.195 0)
       (effects (font (size 1.27 1.27) italic) (justify left) hide)
     )
@@
       (effects (font (size 1.27 1.27)) (justify left))
     )
-    (property "Footprint" "Resistor_THT:R_Axial_DIN0207_L6.3mm_D2.5mm_P2.54mm_Vertical" (at 121.92 179.07 0)
+    (property "Footprint" "Resistor_SMD:R_0402_1005Metric" (at 121.92 179.07 0)
       (effects (font (size 1.27 1.27)) hide)
     )
@@
       (effects (font (size 1.27 1.27)))
     )
-    (property "Footprint" "Resistor_THT:R_Axial_DIN0207_L6.3mm_D2.5mm_P2.54mm_Vertical" (at 203.2 30.48 0)
+    (property "Footprint" "Resistor_SMD:R_0402_1005Metric" (at 203.2 30.48 0)
       (effects (font (size 1.27 1.27)) hide)
     )
@@
       (effects (font (size 1.27 1.27)) (justify left))
     )
-    (property "Footprint" "Package_TO_SOT_THT:TO-92_Inline" (at 217.17 32.385 0)
+    (property "Footprint" "Package_TO_SOT_SMD:SOT-23-3" (at 217.17 32.385 0)
       (effects (font (size 1.27 1.27) italic) (justify left) hide)
     )
@@
       (effects (font (size 1.27 1.27)))
     )
-    (property "Footprint" "Resistor_THT:R_Axial_DIN0207_L6.3mm_D2.5mm_P2.54mm_Vertical" (at 247.65 30.48 0)
+    (property "Footprint" "Resistor_SMD:R_0402_1005Metric" (at 247.65 30.48 0)
       (effects (font (size 1.27 1.27)) hide)
     )
@@
       (effects (font (size 1.27 1.27)) (justify left))
     )
-    (property "Footprint" "" (at 163.83 163.83 0)
+    (property "Footprint" "Package_SO:SOIC-14_3.9x8.7mm_P1.27mm" (at 163.83 163.83 0)
       (effects (font (size 1.27 1.27)) hide)
     )
@@
       (effects (font (size 1.27 1.27)) (justify left))
     )
-    (property "Footprint" "Capacitor_THT:CP_Radial_D5.0mm_P2.00mm" (at 98.7552 44.45 0)
+    (property "Footprint" "Capacitor_SMD:C_1206_3216Metric" (at 98.7552 44.45 0)
       (effects (font (size 1.27 1.27)) hide)
     )
@@
       (effects (font (size 1.27 1.27)))
     )
-    (property "Footprint" "Resistor_THT:R_Axial_DIN0207_L6.3mm_D2.5mm_P2.54mm_Vertical" (at 208.28 99.06 0)
+    (property "Footprint" "Resistor_SMD:R_0402_1005Metric" (at 208.28 99.06 0)
       (effects (font (size 1.27 1.27)) hide)
     )
@@
       (effects (font (size 1.27 1.27)) (justify left))
     )
-    (property "Footprint" "Package_TO_SOT_THT:TO-92_Inline" (at 234.95 32.385 0)
+    (property "Footprint" "Package_TO_SOT_SMD:SOT-23-3" (at 234.95 32.385 0)
       (effects (font (size 1.27 1.27) italic) (justify left) hide)
     )
@@
       (effects (font (size 1.27 1.27)))
     )
-    (property "Footprint" "Resistor_THT:R_Axial_DIN0207_L6.3mm_D2.5mm_P2.54mm_Vertical" (at 77.47 99.06 0)
+    (property "Footprint" "Resistor_SMD:R_0402_1005Metric" (at 77.47 99.06 0)
       (effects (font (size 1.27 1.27)) hide)
     )
@@
       (effects (font (size 1.27 1.27)))
     )
-    (property "Footprint" "Package_DIP:DIP-14_W7.62mm_LongPads" (at 151.13 175.26 0)
+    (property "Footprint" "Package_SO:SOIC-14_3.9x8.7mm_P1.27mm" (at 151.13 175.26 0)
       (effects (font (size 1.27 1.27)) hide)
     )
@@
       (effects (font (size 1.27 1.27)) (justify right))
     )
-    (property "Footprint" "Resistor_THT:R_Axial_DIN0207_L6.3mm_D2.5mm_P2.54mm_Vertical" (at 201.93 133.35 0)
+    (property "Footprint" "Resistor_SMD:R_0402_1005Metric" (at 201.93 133.35 0)
       (effects (font (size 1.27 1.27)) hide)
     )
@@
       (effects (font (size 1.27 1.27)))
     )
-    (property "Footprint" "Resistor_THT:R_Axial_DIN0207_L6.3mm_D2.5mm_P2.54mm_Vertical" (at 167.64 34.29 0)
+    (property "Footprint" "Resistor_SMD:R_0402_1005Metric" (at 167.64 34.29 0)
       (effects (font (size 1.27 1.27)) hide)
     )
@@
       (effects (font (size 1.27 1.27)) (justify left))
     )
-    (property "Footprint" "Package_TO_SOT_THT:TO-92_Inline" (at 154.94 36.195 0)
+    (property "Footprint" "Package_TO_SOT_SMD:SOT-23-3" (at 154.94 36.195 0)
       (effects (font (size 1.27 1.27) italic) (justify left) hide)
     )
@@
       (effects (font (size 1.27 1.27)))
     )
-    (property "Footprint" "Resistor_THT:R_Axial_DIN0207_L6.3mm_D2.5mm_P2.54mm_Vertical" (at 209.55 125.73 0)
+    (property "Footprint" "Resistor_SMD:R_0402_1005Metric" (at 209.55 125.73 0)
       (effects (font (size 1.27 1.27)) hide)
     )
@@
       (effects (font (size 1.27 1.27)) (justify right))
     )
-    (property "Footprint" "Resistor_THT:R_Axial_DIN0207_L6.3mm_D2.5mm_P2.54mm_Vertical" (at 200.66 104.14 0)
+    (property "Footprint" "Resistor_SMD:R_0402_1005Metric" (at 200.66 104.14 0)
       (effects (font (size 1.27 1.27)) hide)
     )
@@
       (effects (font (size 1.27 1.27)) (justify right))
     )
-    (property "Footprint" "Resistor_THT:R_Axial_DIN0207_L6.3mm_D2.5mm_P2.54mm_Vertical" (at 237.49 46.99 0)
+    (property "Footprint" "Resistor_SMD:R_0402_1005Metric" (at 237.49 46.99 0)
       (effects (font (size 1.27 1.27)) hide)
     )
@@
       (effects (font (size 1.27 1.27)) (justify right))
     )
-    (property "Footprint" "Resistor_THT:R_Axial_DIN0207_L6.3mm_D2.5mm_P2.54mm_Vertical" (at 143.51 46.99 0)
+    (property "Footprint" "Resistor_SMD:R_0402_1005Metric" (at 143.51 46.99 0)
       (effects (font (size 1.27 1.27)) hide)
     )
@@
       (effects (font (size 1.27 1.27)))
     )
-    (property "Footprint" "Resistor_THT:R_Axial_DIN0207_L6.3mm_D2.5mm_P2.54mm_Vertical" (at 125.73 34.29 0)
+    (property "Footprint" "Resistor_SMD:R_0402_1005Metric" (at 125.73 34.29 0)
       (effects (font (size 1.27 1.27)) hide)
     )
@@
       (effects (font (size 1.27 1.27)) (justify right))
     )
-    (property "Footprint" "Resistor_THT:R_Axial_DIN0207_L6.3mm_D2.5mm_P2.54mm_Vertical" (at 157.48 46.99 0)
+    (property "Footprint" "Resistor_SMD:R_0402_1005Metric" (at 157.48 46.99 0)
       (effects (font (size 1.27 1.27)) hide)
     )
@@
       (effects (font (size 1.27 1.27)))
     )
-    (property "Footprint" "Resistor_THT:R_Axial_DIN0207_L6.3mm_D2.5mm_P2.54mm_Vertical" (at 172.72 119.38 0)
-      (effects (font (size 1.27 1.27)) hide)
-    )
+    (property "Footprint" "Resistor_SMD:R_0402_1005Metric" (at 172.72 119.38 0)
+      (effects (font (size 1.27 1.27)) hide)
+    )
