File: Pressure-Controlled-Power-Outlet-control-PCB/Pressure-Controlled-Power-Outlet-control-PCB.kicad_sch (KiCad schematic)
At the start: 47 parts, among them J1 pressure sensor, J2 1017514, J3 I2C0 Connector, J4 SPI1 Connector, J5 FanA 5V/24V, J6 FanB 5V/24V, K1 T9GV5L24-24, K2 T9GV5L24-24, M1 Fan_4pin, M2 Fan_4pin, Q1 2N3906, Q2 IRF540N, Q3 IRF540N, Q4 2N3906, Q5 2N3904, Q6 2N3904, Q7 2N3904, Q8 2N3904, U1 Pico, U2 LM324, U3 LF50_TO220

Commit message: hopefully done this PCB
Parts:
- H1, H2, H3, H4: footprint MountingHole:MountingHole_3.2mm_M3_DIN965_Pad -> MountingHole:MountingHole_4.3mm_M4_Pad
Changed lines of the file:
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@@
   (title_block
     (title "Pressure Controlled Power Outlet")
-    (date "2024-07-18")
-    (rev "V1.2.3")
+    (date "2024-07-20")
+    (rev "V1.3.1")
     (company "Brian Banas")
   )
@@
       (effects (font (size 1.27 1.27)))
     )
-    (property "Footprint" "MountingHole:MountingHole_3.2mm_M3_DIN965_Pad" (at 29.21 171.45 0)
+    (property "Footprint" "MountingHole:MountingHole_4.3mm_M4_Pad" (at 29.21 171.45 0)
       (effects (font (size 1.27 1.27)) hide)
     )
@@
       (effects (font (size 1.27 1.27)) (justify left))
     )
-    (property "Footprint" "MountingHole:MountingHole_3.2mm_M3_DIN965_Pad" (at 48.26 171.45 0)
+    (property "Footprint" "MountingHole:MountingHole_4.3mm_M4_Pad" (at 48.26 171.45 0)
       (effects (font (size 1.27 1.27)) hide)
     )
@@
       (effects (font (size 1.27 1.27)) (justify left))
     )
-    (property "Footprint" "MountingHole:MountingHole_3.2mm_M3_DIN965_Pad" (at 49.53 181.61 0)
+    (property "Footprint" "MountingHole:MountingHole_4.3mm_M4_Pad" (at 49.53 181.61 0)
       (effects (font (size 1.27 1.27)) hide)
     )
@@
       (effects (font (size 1.27 1.27)))
     )
-    (property "Footprint" "MountingHole:MountingHole_3.2mm_M3_DIN965_Pad" (at 29.21 181.61 0)
-      (effects (font (size 1.27 1.27)) hide)
-    )
+    (property "Footprint" "MountingHole:MountingHole_4.3mm_M4_Pad" (at 29.21 181.61 0)
+      (effects (font (size 1.27 1.27)) hide)
+    )

Commit message: updated 220µF cap
Parts:
- C1: footprint Capacitor_THT:CP_Radial_D12.5mm_P5.00mm -> Capacitor_THT:CP_Radial_D10.0mm_P5.00mm
Changed lines of the file:
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@@
       (effects (font (size 1.27 1.27)) (justify left))
     )
-    (property "Footprint" "Capacitor_THT:CP_Radial_D12.5mm_P5.00mm" (at 49.2252 43.18 0)
+    (property "Footprint" "Capacitor_THT:CP_Radial_D10.0mm_P5.00mm" (at 49.2252 43.18 0)
       (effects (font (size 1.27 1.27)) hide)
     )
